Commit message: added caster wheels

File: urdf/barista_robot_model.urdf (robot description, URDF)
Before this commit: robot box_bot, 8 links, 7 joints
Links:
- added link back_pitch_link, mass 0.1; collision sphere radius=0.0352; visual sphere radius=0.0352
- added link back_roll_link, mass 0.1; visual cylinder length=0.005 radius=0.0352
- added link back_yaw_link, mass 0.1; visual cylinder length=0.005 radius=0.0352
- added link front_pitch_link, mass 0.1; collision sphere radius=0.0352; visual sphere radius=0.0352
- added link front_roll_link, mass 0.1; visual cylinder length=0.005 radius=0.0352
- added link front_yaw_link, mass 0.1; visual cylinder length=0.005 radius=0.0352
- link chassis: mass 0.5 -> 0.8
- link left_rod: mass 0.001 -> 0.2
- link left_wheel: mass 0.05 -> 0.1
- link right_rod: mass 0.001 -> 0.2
- link right_wheel: mass 0.05 -> 0.1
- link tray_link: mass 0.001 -> 0.5
Joints:
- added joint back_pitch_joint: type continuous, parent back_roll_link, child back_pitch_link, origin xyz=0 0 0 rpy=0 0 0, axis 0 1 0, limit effort=1000.0 velocity=100.0
- added joint back_roll_joint: type continuous, parent back_yaw_link, child back_roll_link, origin xyz=0 0 0 rpy=0 0 0, axis 1 0 0, limit effort=1000.0 velocity=100.0
- added joint back_yaw_joint: type continuous, parent chassis, child back_yaw_link, origin xyz=-0.12 0 -0.075 rpy=0 0 0, axis 0 0 1, limit effort=1000.0 velocity=100.0
- added joint front_pitch_joint: type continuous, parent front_roll_link, child front_pitch_link, origin xyz=0 0 0 rpy=0 0 0, axis 0 1 0, limit effort=1000.0 velocity=100.0
- added joint front_roll_joint: type continuous, parent front_yaw_link, child front_roll_link, origin xyz=0 0 0 rpy=0 0 0, axis 1 0 0, limit effort=1000.0 velocity=100.0
- added joint front_yaw_joint: type continuous, parent chassis, child front_yaw_link, origin xyz=0.12 0 -0.075 rpy=0 0 0, axis 0 0 1, limit effort=1000.0 velocity=100.0

Commit message: added 2 more rods

File: urdf/barista_robot_model.urdf (robot description, URDF)
Before this commit: robot box_bot, 14 links, 13 joints
Links:
- added link left_rod_back, mass 0.2; collision cylinder length=0.220 radius=0.01; visual cylinder length=0.220 radius=0.01
- added link right_rod_back, mass 0.2; collision cylinder length=0.220 radius=0.01; visual cylinder length=0.220 radius=0.01
Joints:
- added joint left_rod_joint_back: type fixed, parent chassis, child left_rod_back, origin xyz=-0.05 -0.14 0.1875 rpy=1.5707 0 0, axis 1 0 0
- added joint right_rod_joint_back: type fixed, parent chassis, child right_rod_back, origin xyz=-0.05 0.14 0.1875 rpy=1.5707 0 0, axis 0 0 1
- joint left_rod_joint: origin xyz=0 -0.14 0.1875 rpy=1.5707 0 0 -> xyz=0.05 -0.14 0.1875 rpy=1.5707 0 0
- joint right_rod_joint: origin xyz=0 0.14 0.1875 rpy=1.5707 0 0 -> xyz=0.05 0.14 0.1875 rpy=1.5707 0 0
