Commit message: fixed rviz configuration not loading and added colours to gazebo

File: xacro/barista_robot_model.urdf.xacro (robot description, xacro)
@@ -1,23 +1,38 @@
 <?xml version="1.0"?>
 <robot xmlns:xacro="http://www.ros.org/wiki/xacro" name = "barista_bot">
+    <xacro:include filename="$(find barista_robot_description)/xacro/standoff.xacro"/>
+    <xacro:include filename="$(find barista_robot_description)/xacro/wheel.xacro"/>
+    <xacro:include filename="$(find barista_robot_description)/xacro/cup_holder_tray.xacro"/>
     <!-- Materials-->
-        <material name="red">
-            <color rgba="1.0 0.0 0.0 1"/>
-        </material>
-        <material name="green_light">
-            <color rgba="0.0 1.0 0.0 1"/>
-        </material>
-        <material name="green_dark">
-            <color rgba="0.0 0.5 0.0 1"/>
-        </material>
-        <material name="blue">
-            <color rgba="0.0 0.0 1.0 1"/>
-        </material>
-        <material name="white">
-            <color rgba="1.0 1.0 1.0 1"/>
-        </material>
-        <material name="black">
-            <color rgba="0.0 0.0 0.0 1"/>
-        </material>
+    <material name="red">
+        <color rgba="1.0 0.0 0.0 1"/>
+    </material>
+    <material name="green_light">
+        <color rgba="0.0 1.0 0.0 1"/>
+    </material>
+    <material name="green_dark">
+        <color rgba="0.0 0.5 0.0 1"/>
+    </material>
+    <material name="blue">
+        <color rgba="0.0 0.0 1.0 1"/>
+    </material>
+    <material name="white">
+        <color rgba="1.0 1.0 1.0 1"/>
+    </material>
+    <material name="black">
+        <color rgba="0.0 0.0 0.0 1"/>
+    </material>
+    <gazebo reference="chassis">
+        <material>Gazebo/Red</material>
+    </gazebo>
+    <gazebo reference="tray_link">
+        <material>Gazebo/Red</material>
+    </gazebo>
+    <gazebo reference="front_yaw_link">
+        <material>Gazebo/Black</material>
+    </gazebo>
+    <gazebo reference="back_yaw_link">
+        <material>Gazebo/Black</material>
+    </gazebo>
   <link name="base_link">
   </link>
@@ -46,5 +61,4 @@
     <child link="chassis" />
   </joint>
-<xacro:include filename="$(find barista_robot_description)/xacro/standoff.xacro"/>
 <joint name="fr_rod_joint" type="fixed">
     <origin rpy="1.5707 0 0" xyz="0.05 0.14 0.1875" />
@@ -71,5 +85,4 @@
     <axis xyz="0 0 1" />
 </joint>
-<xacro:include filename="$(find barista_robot_description)/xacro/wheel.xacro"/>
 <joint name="joint_left_wheel" type="continuous">
     <origin rpy="0 0 0" xyz="0 0.12 -0.075"/>
@@ -88,5 +101,4 @@
     <joint_properties damping="1.0" friction="1.0"/>
   </joint>
-<xacro:include filename="$(find barista_robot_description)/xacro/cup_holder_tray.xacro"/>
 <xacro:arg name="include_laser" default="true"/>
 <xacro:macro name="laser_scanner" params = "include_laser:=true">
