Commit message: added static transform to launch file

File: xacro/blue_barista_robot_model.urdf.xacro (robot description, xacro)
@@ -1,11 +1,8 @@
 <?xml version="1.0"?>
-<robot xmlns:xacro="http://www.ros.org/wiki/xacro" name = "red_barista_bot">
+<robot xmlns:xacro="http://www.ros.org/wiki/xacro" name = "blue_barista_bot">
     <xacro:include filename="$(find barista_robot_description)/xacro/standoff.xacro"/>
     <xacro:include filename="$(find barista_robot_description)/xacro/wheel.xacro"/>
     <xacro:include filename="$(find barista_robot_description)/xacro/cup_holder_tray.xacro"/>
     <!-- Materials-->
-    <material name="main">
-        <color rgba="1.0 0.0 0.0 1"/>
-    </material>
     <material name="green_light">
         <color rgba="0.0 1.0 0.0 1"/>
@@ -14,4 +11,7 @@
         <color rgba="0.0 0.5 0.0 1"/>
     </material>
+    <material name="main">
+        <color rgba="0.0 0.0 1.0 1"/>
+    </material>
     <material name="white">
         <color rgba="1.0 1.0 1.0 1"/>
@@ -21,8 +21,8 @@
     </material>
     <gazebo reference="chassis">
-        <material>Gazebo/Red</material>
+        <material>Gazebo/Blue</material>
     </gazebo>
     <gazebo reference="tray_link">
-        <material>Gazebo/Red</material>
+        <material>Gazebo/Blue</material>
     </gazebo>
     <gazebo reference="front_yaw_link">
@@ -76,5 +76,5 @@
     <axis xyz="0 0 1" />
 </joint>
-<joint name="$bl_rod_joint" type="fixed">
+<joint name="bl_rod_joint" type="fixed">
     <origin rpy="1.5707 0 0" xyz="-0.05 -0.14 0.1875" />
     <parent link="chassis"/>
@@ -137,7 +137,7 @@
         <plugin name="laser" filename="libgazebo_ros_ray_sensor.so">
           <output_type>sensor_msgs/LaserScan</output_type>
-        <ros>
-            <remapping>~/out:=/scan</remapping>
-        </ros>
+          <ros>
+            <remapping>~/out:=blue/scan</remapping>
+          </ros>
         </plugin>
     </sensor>
@@ -149,7 +149,4 @@
   <gazebo>
     <plugin name="box_bot_joint_state" filename="libgazebo_ros_joint_state_publisher.so">
-      <ros>
-          <remapping>~/out:=red/joint_states</remapping>
-      </ros>
       <update_rate>30</update_rate>
       <joint_name>joint_left_wheel</joint_name>
@@ -178,6 +175,6 @@
       <publish_odom>true</publish_odom>
       <publish_odom_tf>true</publish_odom_tf>
-      <odometry_frame>odom</odometry_frame>
-      <robot_base_frame>base_link</robot_base_frame>
+      <odometry_frame>/blue/odom</odometry_frame>
+      <robot_base_frame>/blue/base_link</robot_base_frame>
     </plugin>
   </gazebo>
@@ -189,5 +186,5 @@
           <cylinder length="0.005" radius="0.0206"/>
         </geometry>
-        <material name="blue"/>
+        <material name="main"/>
       </visual>
     <inertial>
@@ -262,5 +259,5 @@
           <cylinder length="0.005" radius="0.0206"/>
         </geometry>
-        <material name="blue"/>
+        <material name="main"/>
       </visual>
       <inertial>

File: xacro/cup_holder_tray.xacro (robot description, xacro)
@@ -8,5 +8,5 @@
         <cylinder length="0.090" radius="0.160"/>
       </geometry>
-      <material name="red"/>
+      <material name="main"/>
     </visual>
     <collision>
